File: Tinkercad Design/Memory Game Arduino Simulation.brd (EAGLE design)
At the start: 56.8 x 53.3 mm, 16 parts

Commit message: Add files via upload
Parts:
- removed R5, R6, R7, R8: 300‎Ω, AUTODESK_CIRCUITS_BREADBOARD:0207/10
- R1, R2, R3, R4: value 300‎Ω -> 220‎Ω
- moved R3 25.4 mm to (5.00, 149.8)
- moved R4 25.4 mm to (5.00, 137.1)
- moved R2 25.4 mm to (5.00, 124.4)
- moved S2 12.7 mm to (5.00, 86.3)
- moved S3 12.7 mm to (5.00, 99.0)
- moved S4 12.7 mm to (5.00, 111.7)
Connections:
- removed net N$3 (its old number): R5.2, S1.2, S1.4
- removed net N$4 (its old number): R7.2, S2.2, S2.4
- removed net N$5 (its old number): R6.2, S3.2, S3.4
- removed net N$6 (its old number): R8.2, S4.2, S4.4
- new net N$10: S1.1, S1.3
- new net N$11: S2.1, S2.3
- new net N$12: S3.1, S3.3
- net N$13: no longer S1.1, S1.3, S2.1, S2.3, S3.1, S3.3
- net N$14: now also S1.2, S1.4, S2.2, S2.4, S3.2, S3.4, S4.2, S4.4; no longer R5.1, R6.1, R7.1, R8.1
